File: Rev A.brd (EAGLE design)
At the start: 130.8 x 100 mm, 96 parts, among them Q101 2N3906, Q102 2N3906, Q103 2N3904, Q104 2N3904, Q105 2N3904, Q106 2N3904, Q107 2N3906, Q108 2N3906, Q109 2N3906, Q110 2N3904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

Commit message: Finished the board layout
Parts:
- moved C201 9.67 mm to (31.8, 35.6), turned to 180 degrees
- moved C202 9.67 mm to (31.8, 86.4), turned to 180 degrees
- moved D103 2.54 mm to (17.8, 90.2)
- moved D104 2.54 mm to (15.2, 90.2)
- turned C203 to 0 degrees
- turned C204 to 0 degrees
- turned R106 to 90 degrees
- turned R108 to 270 degrees
- turned R201 to 180 degrees
Routing:
- net V-: track 0.00 -> 435.7 mm, vias 0 -> 1
- net V+: track 0.00 -> 428.1 mm
- net N$7: track 0.00 -> 141.8 mm
- net SWTIN-: track 0.00 -> 141.5 mm
- net SWTIN+: track 0.00 -> 134.1 mm
- net R_OUT: track 0.00 -> 129.1 mm
- net L_OUT: track 0.00 -> 125.8 mm, vias 0 -> 1
- net N$15: track 0.00 -> 98.3 mm, vias 0 -> 1
- net N$31: track 0.00 -> 62.2 mm, vias 0 -> 1
- net N$41: track 0.00 -> 62.2 mm, vias 0 -> 1
- net N$1: track 0.00 -> 32.3 mm
- net N$36: track 0.00 -> 32.3 mm
- net N$34: track 0.00 -> 29.2 mm
- net N$8: track 0.00 -> 29.2 mm
- net N$29: track 0.00 -> 21.9 mm
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- added copper zone on layer 16, net GND
Other:
- board text added: "Left"
- board text added: "Nathan Campos 2014"
- board text added: "Power12"
- board text added: "Right"
- board text added: "This space was intentionally left blank."
