File: Rev B.brd (EAGLE design)
At the start: 130.8 x 100 mm, 112 parts, among them Q101 BC560C, Q102 BC560C, Q103 BC550B, Q104 BC550B, Q105 BC560C, Q106 BC560C, Q107 BC550B, Q108 BC550B, Q109 BC560C, Q110 BC560C, Q111 BC560C, Q112 BC550B, Q113 BC560C, Q114 BC550B, Q115 2N3904, Q116 2N3906, Q117 2N3904, Q118 2N3906, Q119 TIP42C, Q120 TIP41C, Q121 TIP42C, Q122 TIP41C

Commit message: Finished routing one side
Parts:
- removed C107, C108: 2.2uF, rcl:E2-5
- removed C109, C110: 100pF, rcl:C050-050X075
- removed C111, C112: 100n, rcl:C075-042X103
- removed D107, D108, D109, D110, D111, D112: 1N4148DO35-7, diode:DO35-7
- removed KK103, KK104: SK129-PAD, heatsink:SK129
- removed L_IN+, L_IN-, L_SPK+, L_SPK-: PIN2F061.100, con-faston:F061.100
- removed Q112, Q114: BC550B, transistor-npn:TO92-EBC
- removed Q113: BC560C, transistor-pnp:TO92-EBC
- removed Q115, Q117: 2N3904, transistor-npn:TO92
- removed Q116, Q118: 2N3906, transistor-pnp:TO92
- removed Q119, Q121: TIP42C, transistor-power:TO220AV
- removed Q120, Q122: TIP41C, transistor-power:TO220AV
- removed R117, R118: 10kΩ, rcl:0207/10
- removed R119, R120: 4.7kΩ, rcl:0207/10
- removed R121, R122: 560, rcl:0207/10
- removed R123, R124, R125, R126: 1kΩ, rcl:0207/10
- removed R127, R128, R129, R130: 0.33Ω, rcl:0309/12
- removed R131, R132: 10Ω, resistor-power:MNS-5
- removed U$8: (no value), dicons:ICON_AC
- added C205: 100nF, rcl:C025-025X050
- added U$9: (no value), dicons:ICON_EXL-S
- added UNITY: (no value), jumper:JP1
- C102: value 4.7uF -> 10nF; device rcl:C225-113X268 -> rcl:C025-025X050
- C103: value 10nF -> 220uF; device rcl:C025-025X050 -> rcl:E3,5-8
- C104: value 10nF -> 2.2uF; device rcl:C025-025X050 -> rcl:E2-5
- C105: value 220uF -> 100pF; device rcl:E5-10,5 -> rcl:C050-050X075
- C106: value 220uF -> 100n; device rcl:E5-10,5 -> rcl:C075-042X103
- C201, C202: value 100nF -> 2200uF; device rcl:C025-025X050 -> rcl:E5-10,5
- C203, C204: value 4700uF -> 2200uF; device rcl:E7,5-16 -> rcl:E5-10,5
- Q102: value BC560C -> BC550B; device transistor-pnp:TO92-EBC -> transistor-npn:TO92-EBC
- Q103: value BC550B -> BC560C; device transistor-npn:TO92-EBC -> transistor-pnp:TO92-EBC
- Q108: value BC550B -> 2N3904; device transistor-npn:TO92-EBC -> transistor-npn:TO92
- Q109: value BC560C -> 2N3906; device transistor-pnp:TO92-EBC -> transistor-pnp:TO92
- Q110: value BC560C -> TIP42C; device transistor-pnp:TO92-EBC -> transistor-power:TO220AV
- Q111: value BC560C -> TIP41C; device transistor-pnp:TO92-EBC -> transistor-power:TO220AV
- R102: value 10kΩ -> 100Ω
- R103: value 100Ω -> 22Ω
- R104: value 100Ω -> 56Ω
- R105: value 22Ω -> 100Ω
- R106: value 56Ω -> 22Ω
- R107: value 22Ω -> 56Ω
- R108: value 56Ω -> 560Ω
- R109: value 100Ω -> 10kΩ
- R110: value 100Ω -> 4.7kΩ
- R111: value 22Ω -> 560
- R112: value 56Ω -> 1kΩ
- R113: value 22Ω -> 1kΩ
- R114: value 56Ω -> 0.33Ω; device rcl:0207/10 -> rcl:0309/12
- R115: value 560Ω -> 0.33Ω; device rcl:0207/10 -> rcl:0309/12
- R116: value 560Ω -> 10Ω; device rcl:0207/10 -> rcl:0617V
- U$2: device dicons:ICON_SPEAKER -> dicons:ICON_GND2
- U$3: device dicons:ICON_TEMP -> dicons:ICON_PLUS
- U$4: device dicons:ICON_TEMP -> dicons:ICON_MINUS
- moved SWT_OUT- 322.0 mm to (-10.2, -246.4), turned to 0 degrees
- moved SWT_IN- 319.4 mm to (-10.2, -228.6), turned to 0 degrees
- moved SWT_OUT+ 312.7 mm to (-10.2, -237.5), turned to 0 degrees
- moved SWT_IN+ 310.2 mm to (-10.2, -219.7), turned to 0 degrees
- moved R110 280.9 mm to (21.6, 40.6), turned to 90 degrees
- moved R201 280.3 mm to (-8.89, -214.6), turned to 0 degrees
- moved R116 275.1 mm to (99.1, 25.4), turned to 180 degrees
- moved R108 265.5 mm to (40.6, 25.4), turned to 180 degrees
- moved R114 264.6 mm to (63.5, 24.1), turned to 90 degrees
- moved D104 262.8 mm to (33.0, 38.1), turned to 90 degrees
- moved R107 262.0 mm to (11.4, 21.6), turned to 270 degrees
- moved R104 261.8 mm to (14.0, 21.6), turned to 270 degrees
- moved D103 260.7 mm to (30.5, 38.1), turned to 270 degrees
- moved R113 259.8 mm to (80.0, 24.1), turned to 90 degrees
- moved Q106 247.7 mm to (25.4, 40.6), turned to 270 degrees
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Connections:
- removed net L_OUT: D111.A, D112.C, L_SPK+.A1, L_SPK+.A2, R118.2, R129.1, R130.2, R132.2
- removed net N$15: C102.1, L_IN+.A1, L_IN+.A2
- removed net N$17: Q104.B, Q108.B, Q108.C, Q110.C
- removed net N$21: C102.2, R102.2, R104.1
- removed net N$22: Q110.E, R113.1
- removed net N$23: C110.1, Q102.C, Q104.C, Q114.B
- removed net N$24 (its old number): D105.C, D106.A
- removed net N$25: D107.C, D108.A
- removed net N$30: D107.A, Q113.C, Q117.2
- removed net N$33: Q117.1, Q121.B, R125.1
- removed net N$34: Q117.3, Q121.C, R129.2
- removed net N$35: Q118.1, Q122.B, R126.2
- removed net N$36: Q118.3, Q122.C, R130.1
- removed net N$37: C110.2, D108.C, Q114.C, Q118.2
- removed net N$38: Q110.B, R116.2, R118.1
- removed net N$39: C108.+, D104.C, Q106.B, Q113.B, R120.2
- removed net N$41: Q113.E, R122.1
- removed net N$42: C112.1, R132.1
- removed net N$43: Q102.E, R107.1
- removed net N$44: Q106.C, R107.2, R113.2
- removed net N$45: Q106.E, R110.1
- removed net N$46: C104.1, Q102.B, R104.2
- removed net N$47: C106.+, R116.1
- removed net N$48: Q104.E, R108.2
- removed net N$49: Q108.E, R114.2
- net GND: now also C102.2, C103.-, C104.-, C106.2, C201.+, C202.+, C203.-, R110.1; no longer C103.2, C104.2, C105.-, C106.-, C107.-, C108.-, C111.2, C112.2, C203.+, L_IN-.A1, L_IN-.A2, L_SPK-.A1, L_SPK-.A2, R102.1, R119.1, R120.1
- net N$1: now also D103.A, Q106.C, Q108.2; no longer D105.A, Q111.C, Q115.2
- net N$11: now also Q106.E, R111.1; no longer Q111.E, R121.1
- net N$12: now also C103.+, R108.1; no longer C105.+, R115.1
- net N$13: now also Q102.E, R104.2; no longer Q103.E, R106.2
- net N$14: now also Q104.E, R107.2; no longer Q107.E, R112.2
- net N$16: now also C106.1, R116.1; no longer C111.1, R131.1
- net N$18: now also R103.1; no longer R105.1
- net N$19: now also Q103.C, R103.2, R106.2; no longer Q105.C, R105.2, R111.2
- net N$2: now also Q105.E, R106.1; no longer Q109.E, R111.1
- net N$20: now also Q103.E, R105.1; no longer Q105.E, R109.1
- net N$26: now also Q108.1, Q110.B, R112.1; no longer Q115.1, Q119.B, R123.1
- net N$27: now also Q109.1, Q111.B, R113.2; no longer Q116.1, Q120.B, R124.2
- net N$28: now also Q109.3, Q111.C, R115.1; no longer Q116.3, Q120.C, R128.1
- net N$29: now also Q108.3, Q110.C, R114.2; no longer Q115.3, Q119.C, R127.2
- net N$3: now also Q102.B, Q104.B, Q104.C, Q105.C; no longer Q103.B, Q107.B, Q107.C, Q109.C
- net N$31: now also C105.2, D104.C, Q107.C, Q109.2; no longer C109.2, D106.C, Q112.C, Q116.2
- net N$32: now also Q105.B, R108.2, R109.1, UNITY.1; no longer Q109.B, R115.2, R117.1
- net N$4: now also C102.1, R102.2; no longer C103.1, R103.2
- net N$5: now also R102.1; no longer R103.1
- net N$6: now also C104.+, Q103.B, Q106.B, R110.2; no longer C107.+, Q105.B, Q111.B, R119.2
- net N$8: now also C105.1, Q102.C, Q107.B; no longer C109.1, Q103.C, Q112.B
- net R_OUT: now also D105.A, D106.C, R109.2, R114.1, R115.2, R116.2, UNITY.2; no longer D109.A, D110.C, R117.2, R127.1, R128.2, R131.2
- net V+: now also C203.+, C205.1, D105.C, Q110.E, R105.2, R111.2, R112.2; no longer C201.1, C202.1, D103.A, D109.C, D111.C, Q119.E, Q121.E, R109.2, R110.2, R121.2, R122.2, R123.2, R125.2
- net V-: now also C201.-, C202.-, C205.2, D106.A, Q107.E, Q111.E, R104.1, R107.1, R113.1; no longer C201.2, C202.2, C203.-, D110.A, D112.A, Q112.E, Q114.E, Q120.E, Q122.E, R106.1, R108.1, R112.1, R114.1, R124.1, R126.1
Routing:
- net SWTIN-: track 140.8 -> 0.00 mm
- net SWTIN+: track 131.8 -> 5.00 mm
- net V+: track 8.07 -> 110.2 mm
- net N$7: track 5.00 -> 104.4 mm
- net R_OUT: track 7.54 -> 104.7 mm
- net V-: track 5.00 -> 82.4 mm
- net N$31: track 0.00 -> 61.3 mm
- net N$8: track 0.00 -> 44.3 mm
- net N$1: track 0.00 -> 43.5 mm
- net N$14: track 0.00 -> 39.7 mm
- net N$6: track 9.94 -> 36.4 mm
- net N$13: track 0.00 -> 21.4 mm
- net N$32: track 2.54 -> 22.6 mm
- net N$28: track 0.00 -> 19.4 mm
- net N$29: track 0.00 -> 19.4 mm
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Other:
- board text removed: "Left"
- board text removed: "This space was intentionally left blank."
