File: Rev B (Before Duplication).brd (EAGLE design)
At the start: 130.8 x 100 mm, 121 parts, among them Q1 BC560C, Q10 TIP42C, Q11 TIP41C, Q12 BC560C, Q13 BC560C, Q14 2N3906, Q15 BC560C, Q16 BC550B, Q17 BC550B, Q18 2N3904, Q19 BC550B, Q2 BC550B, Q20 TIP41C, Q21 TIP42C, Q22 BC560C, Q3 BC560C, Q4 BC550B, Q5 BC560C, Q6 BC560C, Q7 BC550B, Q8 2N3904, Q9 2N3906

Commit message: Rev B
Parts:
- removed C1, C13: 4.7uF, rcl:C225-113X268
- removed C11, C18: 100nF, rcl:C025-025X050
- removed C12, C5: 100pF, rcl:C050-050X075
- removed C14, C6: 100n, rcl:C075-042X103
- removed C15, C2: 10nF, rcl:C025-025X050
- removed C16, C4: 2.2uF, rcl:E2-5
- removed C17, C3: 220uF, rcl:E3,5-8
- removed D1, D10, D11, D12, D2, D3, D4, D5, D6, D7, D8, D9: 1N4148DO35-7, diode:DO35-7
- removed KK1, KK2, KK3, KK4: SK129-PAD, heatsink:SK129
- removed L_IN+, L_IN-, L_SPK+, L_SPK-: PIN2F061.100, con-faston:F061.100
- removed Q1, Q12, Q13, Q15, Q22, Q3, Q5, Q6: BC560C, transistor-pnp:TO92-EBC
- removed Q10, Q21: TIP42C, transistor-power:TO220AV
- removed Q11, Q20: TIP41C, transistor-power:TO220AV
- removed Q14, Q9: 2N3906, transistor-pnp:TO92
- removed Q16, Q17, Q19, Q2, Q4, Q7: BC550B, transistor-npn:TO92-EBC
- removed Q18, Q8: 2N3904, transistor-npn:TO92
- removed R10, R17, R25: 4.7kΩ, rcl:0207/10
- removed R11, R26: 560, rcl:0207/10
- removed R12, R13, R19, R20: 1kΩ, rcl:0207/10
- removed R14, R15, R23, R24: 0.33Ω, rcl:0309/12
- removed R16, R27: 10Ω, rcl:0617V
- removed R18, R22, R9: 10kΩ, rcl:0207/10
- removed R2, R30, R31, R5: 100Ω, rcl:0207/10
- removed R21: 560Ω, rcl:0207/10
- removed R28, R29, R3, R6: 22Ω, rcl:0207/10
- removed R32, R33, R4, R7: 56Ω, rcl:0207/10
- removed U$10, U$11: (no value), dicons:ICON_TEMP
- removed U$12: (no value), dicons:ICON_AC
- removed U$13: (no value), dicons:ICON_EXL-S
- removed U$8: (no value), dicons:ICON_SPEAKER
- removed UNITY1: (no value), jumper:JP1
- added C101: 4.7uF, rcl:C225-113X268
- added C102: 10nF, rcl:C025-025X050
- added C103: 220uF, rcl:E3,5-8
- added C104: 2.2uF, rcl:E2-5
- added C105: 100pF, rcl:C050-050X075
- added C106: 100n, rcl:C075-042X103
- added C205: 100nF, rcl:C025-025X050
- added D101, D102, D103, D104, D105, D106: 1N4148DO35-7, diode:DO35-7
- added KK101, KK102: SK129-PAD, heatsink:SK129
- added Q101, Q103, Q105, Q106: BC560C, transistor-pnp:TO92-EBC
- added Q102, Q104, Q107: BC550B, transistor-npn:TO92-EBC
- added Q108: 2N3904, transistor-npn:TO92
- added Q109: 2N3906, transistor-pnp:TO92
- added Q110: TIP42C, transistor-power:TO220AV
- added Q111: TIP41C, transistor-power:TO220AV
- added R101: 10kΩ, rcl:0207/10
- added R103, R106: 22Ω, rcl:0207/10
- added R104, R107: 56Ω, rcl:0207/10
- added R105: 100Ω, rcl:0207/10
- added R108: 560Ω, rcl:0207/10
- added R110, R201: 4.7kΩ, rcl:0207/10
- added R111: 560, rcl:0207/10
- added R112, R113: 1kΩ, rcl:0207/10
- added R114, R115: 0.33Ω, rcl:0309/12
- added R116: 10Ω, rcl:0617V
- R102: value 10kΩ -> 100Ω
- R109: value 560Ω -> 10kΩ
- moved SWT_OUT- 320.6 mm to (-10.2, -246.4), turned to 0 degrees
- moved SWT_IN- 318.1 mm to (-10.2, -228.6), turned to 0 degrees
- moved SWT_OUT+ 311.5 mm to (-10.2, -237.5), turned to 0 degrees
- moved SWT_IN+ 308.9 mm to (-10.2, -219.7), turned to 0 degrees
- moved ON 111.8 mm to (5.08, -5.08), turned to 0 degrees
- moved U$2 30.5 mm to (125.7, 19.1)
- moved GND1_ 30.5 mm to (124.5, 26.7)
- moved GND2_ 30.5 mm to (124.5, 11.4)
- moved PWR+ 30.5 mm to (118.1, 26.7)
- moved PWR- 30.5 mm to (118.1, 11.4)
- moved U$3 30.5 mm to (118.1, 20.3)
- moved U$4 30.5 mm to (118.1, 17.8)
- moved U$9 2.54 mm to (71.1, 24.1)
- moved UNITY 2.54 mm to (40.6, 30.5)
- moved U$7 2.54 mm to (108.0, 15.2)
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- renumbered C10 to C204, C7 to C201, C8 to C202, C9 to C203, R1 to R102, R8 to R109
Connections:
- removed net L_OUT: D10.C, D7.A, L_SPK+.A1, L_SPK+.A2, R22.2, R23.1, R24.2, R27.2, UNITY1.2
- removed net N$15: Q15.C, Q16.B, Q16.C, Q19.B
- removed net N$17: C13.2, R18.2, R31.1
- removed net N$21: Q15.E, R28.1
- removed net N$22: C12.1, Q13.C, Q17.B, Q19.C
- removed net N$23: D8.A, D9.C
- removed net N$25: D9.A, Q12.C, Q18.2
- removed net N$30: Q18.1, Q21.B, R19.1
- removed net N$33: Q18.3, Q21.C, R23.2
- removed net N$34: Q14.1, Q20.B, R20.2
- removed net N$35: Q14.3, Q20.C, R24.1
- removed net N$36: C12.2, D8.C, Q14.2, Q17.C
- removed net N$37: Q15.B, R21.2, R22.1, UNITY1.1
- removed net N$38: C13.1, L_IN+.A1, L_IN+.A2
- removed net N$39: C16.+, D11.C, Q12.B, Q22.B, R25.2
- removed net N$40: D11.A, D12.C
- removed net N$41: Q12.E, R26.1
- removed net N$42: C14.1, R27.1
- removed net N$43: Q13.E, R29.1
- removed net N$44: Q22.C, R28.2, R29.2
- removed net N$45: Q22.E, R30.1
- removed net N$46: C15.1, Q13.B, R31.2
- removed net N$47: C17.+, R21.1
- removed net N$48: Q19.E, R32.2
- removed net N$49: Q16.E, R33.2
- net GND: now also C102.2, C103.-, C104.-, C106.2, R101.1, R110.1; no longer C14.2, C15.2, C16.-, C17.-, C2.2, C3.-, C4.-, C6.2, L_IN-.A1, L_IN-.A2, L_SPK-.A1, L_SPK-.A2, R10.1, R102.1, R18.1, R25.1
- net N$1: now also D103.A, Q106.C, Q108.2; no longer D3.A, Q6.C, Q8.2
- net N$10: now also R201.2; no longer R17.2
- net N$11: now also Q106.E, R111.1; no longer Q6.E, R11.1
- net N$12: now also C103.+, R108.1; no longer C3.+, R109.1
- net N$13: now also Q102.E, R104.2; no longer Q2.E, R4.2
- net N$14: now also Q104.E, R107.2; no longer Q4.E, R7.2
- net N$16: now also C106.1, R116.1; no longer C6.1, R16.1
- net N$18: now also Q101.E, R103.1; no longer Q1.E, R3.1
- net N$19: now also Q103.C, R103.2, R106.2; no longer Q3.C, R3.2, R6.2
- net N$2: now also Q105.E, R106.1; no longer Q5.E, R6.1
- net N$20: now also Q103.E, R105.1; no longer Q3.E, R5.1
- net N$24: now also D103.C, D104.A; no longer D3.C, D4.A
- net N$26: now also Q108.1, Q110.B, R112.1; no longer Q10.B, Q8.1, R12.1
- net N$27: now also Q109.1, Q111.B, R113.2; no longer Q11.B, Q9.1, R13.2
- net N$28: now also Q109.3, Q111.C, R115.1; no longer Q11.C, Q9.3, R15.1
- net N$29: now also Q108.3, Q110.C, R114.2; no longer Q10.C, Q8.3, R14.2
- net N$3: now also Q102.B, Q104.B, Q104.C, Q105.C; no longer Q2.B, Q4.B, Q4.C, Q5.C
- net N$31: now also C105.2, D104.C, Q107.C, Q109.2; no longer C5.2, D4.C, Q7.C, Q9.2
- net N$32: now also Q105.B, R108.2, R109.1; no longer Q5.B, R109.2, R9.1
- net N$4: now also C102.1, Q101.B, R102.2; no longer C2.1, Q1.B, R2.2
- net N$5: now also C101.2, R101.2, R102.1; no longer C1.2, R102.2, R2.1
- net N$6: now also C104.+, D102.C, Q103.B, Q106.B, R110.2; no longer C4.+, D2.C, Q3.B, Q6.B, R10.2
- net N$7: now also C101.1; no longer C1.1
- net N$8: now also C105.1, Q101.C, Q102.C, Q107.B; no longer C5.1, Q1.C, Q2.C, Q7.B
- net N$9: now also D101.C, D102.A; no longer D1.C, D2.A
- net R_OUT: now also D105.A, D106.C, R109.2, R114.1, R115.2, R116.2; no longer D5.A, D6.C, R14.1, R15.2, R16.2, R9.2
- net V+: now also C205.1, D101.A, D105.C, Q110.E, R105.2, R111.2, R112.2; no longer C11.1, C18.1, D1.A, D12.A, D5.C, D7.C, Q10.E, Q21.E, R11.2, R12.2, R19.2, R26.2, R30.2, R5.2
- net V-: now also C205.2, D106.A, Q107.E, Q111.E, R104.1, R107.1, R113.1, R201.1; no longer C11.2, C18.2, D10.A, D6.A, Q11.E, Q17.E, Q20.E, Q7.E, R13.1, R17.1, R20.1, R32.1, R33.1, R4.1, R7.1
Routing:
- net V-: track 355.5 -> 82.4 mm
- net V+: track 360.4 -> 110.2 mm, vias 8 -> 0
- net SWTIN-: track 179.4 -> 0.00 mm
- net SWTIN+: track 164.0 -> 5.00 mm
- net L_OUT: track 104.0 -> 0.00 mm
- net N$38: track 102.9 -> 0.00 mm, vias 2 -> 0
- net N$36: track 61.3 -> 0.00 mm
- net N$22: track 44.3 -> 0.00 mm
- net N$25: track 43.5 -> 0.00 mm
- net N$39: track 41.5 -> 0.00 mm
- net N$49: track 39.7 -> 0.00 mm
- net GND: track 22.9 -> 0.00 mm, vias 12 -> 0
- net N$37: track 22.6 -> 0.00 mm
- net N$48: track 21.4 -> 0.00 mm
- net N$35: track 19.4 -> 0.00 mm
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- removed copper zone on layer 16, net GND
Other:
- board text removed: "Left"
- board text removed: "Serial #"
- board text removed: "UNITY"
