File: Rev B.sch (EAGLE design)
At the start: 104 parts, among them Q101 BC560C, Q102 BC560C, Q103 BC550B, Q104 BC550B, Q105 BC560C, Q106 BC560C, Q107 BC550B, Q108 BC550B, Q109 BC560C, Q110 BC560C, Q111 BC560C, Q112 BC550B, Q113 BC560C, Q114 BC550B, Q115 2N3904, Q116 2N3906, Q117 2N3904, Q118 2N3906, Q119 TIP42C, Q120 TIP41C, Q121 TIP42C, Q122 TIP41C

Commit message: Finished routing one side
Parts:
- removed C107, C108: 2.2uF, rcl:CPOL-EUE2-5
- removed C109, C110: 100pF, rcl:C-EU050-050X075
- removed C111, C112: 100n, rcl:C-EU075-042X103
- removed D107, D108, D109, D110, D111, D112: 1N4148DO35-7, diode:1N4148DO35-7
- removed KK103, KK104: SK129-PAD, heatsink:SK129-PAD
- removed L_IN+, L_IN-, L_SPK+, L_SPK-: PIN2F061.100, con-faston:PIN2F061.100
- removed Q112, Q114: BC550B, transistor-npn:BC550B
- removed Q113: BC560C, transistor-pnp:BC560C
- removed Q115, Q117: 2N3904, transistor-npn:2N3904
- removed Q116, Q118: 2N3906, transistor-pnp:2N3906
- removed Q119, Q121: TIP42C, transistor-power:TIP42C
- removed Q120, Q122: TIP41C, transistor-power:TIP41C
- removed R117, R118: 10kΩ, rcl:R-EU_0207/10
- removed R119, R120: 4.7kΩ, rcl:R-EU_0207/10
- removed R121, R122: 560, rcl:R-EU_0207/10
- removed R123, R124, R125, R126: 1kΩ, rcl:R-EU_0207/10
- removed R127, R128, R129, R130: 0.33Ω, rcl:R-EU_0309/12
- removed R131, R132: 10Ω, resistor-power:RMNS-5
- added C205: 100nF, rcl:C-EU025-025X050
- added UNITY: (no value), jumper:JP1E
- C102: value 4.7uF -> 10nF; device rcl:C-EU225-113X268 -> rcl:C-EU025-025X050
- C103: value 10nF -> 220uF; device rcl:C-EU025-025X050 -> rcl:CPOL-EUE3.5-8
- C104: value 10nF -> 2.2uF; device rcl:C-EU025-025X050 -> rcl:CPOL-EUE2-5
- C105: value 220uF -> 100pF; device rcl:CPOL-EUE5-10.5 -> rcl:C-EU050-050X075
- C106: value 220uF -> 100n; device rcl:CPOL-EUE5-10.5 -> rcl:C-EU075-042X103
- C201, C202: value 100nF -> 2200uF; device rcl:C-EU025-025X050 -> rcl:CPOL-EUE5-10.5
- C203, C204: value 4700uF -> 2200uF; device rcl:CPOL-EUE7.5-16 -> rcl:CPOL-EUE5-10.5
- Q102: value BC560C -> BC550B; device transistor-pnp:BC560C -> transistor-npn:BC550B
- Q103: value BC550B -> BC560C; device transistor-npn:BC550B -> transistor-pnp:BC560C
- Q108: value BC550B -> 2N3904; device transistor-npn:BC550B -> transistor-npn:2N3904
- Q109: value BC560C -> 2N3906; device transistor-pnp:BC560C -> transistor-pnp:2N3906
- Q110: value BC560C -> TIP42C; device transistor-pnp:BC560C -> transistor-power:TIP42C
- Q111: value BC560C -> TIP41C; device transistor-pnp:BC560C -> transistor-power:TIP41C
- R102: value 10kΩ -> 100Ω
- R103: value 100Ω -> 22Ω
- R104: value 100Ω -> 56Ω
- R105: value 22Ω -> 100Ω
- R106: value 56Ω -> 22Ω
- R107: value 22Ω -> 56Ω
- R108: value 56Ω -> 560Ω
- R109: value 100Ω -> 10kΩ
- R110: value 100Ω -> 4.7kΩ
- R111: value 22Ω -> 560
- R112: value 56Ω -> 1kΩ
- R113: value 22Ω -> 1kΩ
- R114: value 56Ω -> 0.33Ω; device rcl:R-EU_0207/10 -> rcl:R-EU_0309/12
- R115: value 560Ω -> 0.33Ω; device rcl:R-EU_0207/10 -> rcl:R-EU_0309/12
- R116: value 560Ω -> 10Ω; device rcl:R-EU_0207/10 -> rcl:R-EU_0617/5V
Connections:
- removed net L_OUT: D111.A, D112.C, L_SPK+.1, R118.2, R129.1, R130.2, R132.2
- removed net N$15: C102.1, L_IN+.1
- removed net N$17: Q104.B, Q108.B, Q108.C, Q110.C
- removed net N$21: C102.2, R102.2, R104.1
- removed net N$22: Q110.E, R113.1
- removed net N$23: C110.1, Q102.C, Q104.C, Q114.B
- removed net N$24 (its old number): D105.C, D106.A
- removed net N$25: D107.C, D108.A
- removed net N$30: D107.A, Q113.C, Q117.B
- removed net N$33: Q117.C, Q121.B, R125.1
- removed net N$34: Q117.E, Q121.C, R129.2
- removed net N$35: Q118.C, Q122.B, R126.2
- removed net N$36: Q118.E, Q122.C, R130.1
- removed net N$37: C110.2, D108.C, Q114.C, Q118.B
- removed net N$38: Q110.B, R116.2, R118.1
- removed net N$39: C108.+, D104.C, Q106.B, Q113.B, R120.2
- removed net N$41: Q113.E, R122.1
- removed net N$42: C112.1, R132.1
- removed net N$43: Q102.E, R107.1
- removed net N$44: Q106.C, R107.2, R113.2
- removed net N$45: Q106.E, R110.1
- removed net N$46: C104.1, Q102.B, R104.2
- removed net N$47: C106.+, R116.1
- removed net N$48: Q104.E, R108.2
- removed net N$49: Q108.E, R114.2
- net GND: now also C102.2, C103.-, C104.-, C106.2, C201.+, C202.+, C203.-, R110.1; no longer C103.2, C104.2, C105.-, C106.-, C107.-, C108.-, C111.2, C112.2, C203.+, L_IN-.1, L_SPK-.1, R102.1, R119.1, R120.1
- net N$1: now also D103.A, Q106.C, Q108.B; no longer D105.A, Q111.C, Q115.B
- net N$11: now also Q106.E, R111.1; no longer Q111.E, R121.1
- net N$12: now also C103.+, R108.1; no longer C105.+, R115.1
- net N$13: now also Q102.E, R104.2; no longer Q103.E, R106.2
- net N$14: now also Q104.E, R107.2; no longer Q107.E, R112.2
- net N$16: now also C106.1, R116.1; no longer C111.1, R131.1
- net N$18: now also R103.1; no longer R105.1
- net N$19: now also Q103.C, R103.2, R106.2; no longer Q105.C, R105.2, R111.2
- net N$2: now also Q105.E, R106.1; no longer Q109.E, R111.1
- net N$20: now also Q103.E, R105.1; no longer Q105.E, R109.1
- net N$26: now also Q108.C, Q110.B, R112.1; no longer Q115.C, Q119.B, R123.1
- net N$27: now also Q109.C, Q111.B, R113.2; no longer Q116.C, Q120.B, R124.2
- net N$28: now also Q109.E, Q111.C, R115.1; no longer Q116.E, Q120.C, R128.1
- net N$29: now also Q108.E, Q110.C, R114.2; no longer Q115.E, Q119.C, R127.2
- net N$3: now also Q102.B, Q104.B, Q104.C, Q105.C; no longer Q103.B, Q107.B, Q107.C, Q109.C
- net N$31: now also C105.2, D104.C, Q107.C, Q109.B; no longer C109.2, D106.C, Q112.C, Q116.B
- net N$32: now also Q105.B, R108.2, R109.1, UNITY.1; no longer Q109.B, R115.2, R117.1
- net N$4: now also C102.1, R102.2; no longer C103.1, R103.2
- net N$5: now also R102.1; no longer R103.1
- net N$6: now also C104.+, Q103.B, Q106.B, R110.2; no longer C107.+, Q105.B, Q111.B, R119.2
- net N$8: now also C105.1, Q102.C, Q107.B; no longer C109.1, Q103.C, Q112.B
- net R_OUT: now also D105.A, D106.C, R109.2, R114.1, R115.2, R116.2, UNITY.2; no longer D109.A, D110.C, R117.2, R127.1, R128.2, R131.2
- net V+: now also C203.+, C205.1, D105.C, Q110.E, R105.2, R111.2, R112.2; no longer C201.1, C202.1, D103.A, D109.C, D111.C, Q119.E, Q121.E, R109.2, R110.2, R121.2, R122.2, R123.2, R125.2
- net V-: now also C201.-, C202.-, C205.2, D106.A, Q107.E, Q111.E, R104.1, R107.1, R113.1; no longer C201.2, C202.2, C203.-, D110.A, D112.A, Q112.E, Q114.E, Q120.E, Q122.E, R106.1, R108.1, R112.1, R114.1, R124.1, R126.1
Other:
- moved on the sheet: C102, C203, C204, D103, D104, D105, D106, KK101, KK102, ON, Q104, Q105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

Commit message: Rev B
Parts:
- removed KK101, KK102: SK129-PAD, heatsink:SK129-PAD
- added KK1, KK2: SK129-PAD, heatsink:SK129-PAD
- renumbered C101 to C1, C102 to C2, C103 to C3, C104 to C4, C105 to C5, C106 to C6, C201 to C7, C202 to C8, C203 to C9, C204 to C10, C205 to C11, D101 to D1, D102 to D2, D103 to D3, D104 to D4, D105 to D5, D106 to D6, Q101 to Q1, Q102 to Q2, Q103 to Q3, Q104 to Q4, Q105 to Q5, Q106 to Q6, Q107 to Q7, Q108 to Q8, Q109 to Q9, Q110 to Q10, Q111 to Q11, R101 to R1, R102 to R2, R103 to R3, R104 to R4, R105 to R5, R106 to R6, R107 to R7, R108 to R8, R109 to R9, R110 to R10, R111 to R11, R112 to R12, R113 to R13, R114 to R14, R115 to R15, R116 to R16, R201 to R17
